File: scupper84.kicad_pcb (KiCad board)
At the start: 2 copper layers, 276.9 x 127.3 mm, 258 parts, among them K1 PG1350, K10 PG1350, K11 PG1350, K12 PG1350, K13 PG1350, K14 PG1350, K15 PG1350, K16 PG1350, K17 PG1350, K18 PG1350, K19 PG1350, K2 PG1350, K20 PG1350, K21 PG1350, K22 PG1350, K23 PG1350, K24 PG1350, K25 PG1350, K26 PG1350, K27 PG1350, K28 PG1350, K29 PG1350, K3 PG1350, K30 PG1350, K31 PG1350, K32 PG1350, K33 PG1350, K34 PG1350, K35 PG1350, K36 PG1350, K37 PG1350, K38 PG1350, K39 PG1350, K4 PG1350, K40 PG1350, K41 PG1350, K42 PG1350, K43 PG1350, K44 PG1350, K45 PG1350, K46 PG1350, K47 PG1350, K48 PG1350, K49 PG1350, K5 PG1350, K50 PG1350, K51 PG1350, K52 PG1350, K53 PG1350, K54 PG1350, K55 PG1350, K56 PG1350, K57 PG1350, K58 PG1350, K59 PG1350, K6 PG1350, K60 PG1350, K61 PG1350, K62 PG1350, K63 PG1350, K64 PG1350, K65 PG1350, K66 PG1350, K67 PG1350, K68 PG1350, K69 PG1350, K7 PG1350, K70 PG1350, K71 PG1350, K72 PG1350, K73 PG1350, K74 PG1350, K75 PG1350, K76 PG1350, K77 PG1350, K78 PG1350, K79 PG1350, K8 PG1350, K80 PG1350, K81 PG1350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

Commit message: Arranging diodes.
Parts:
- moved D84 205.0 mm to (273.0, 16.5), turned to 90 degrees
- moved D31 201.6 mm to (30.0, 16.5), turned to 90 degrees
- moved D32 200.9 mm to (35.9, 16.5), turned to 90 degrees
- moved D33 200.4 mm to (41.8, 16.5), turned to 90 degrees
- moved D36 200.4 mm to (59.6, 16.5), turned to 90 degrees
- moved D34 200.2 mm to (47.8, 16.5), turned to 90 degrees
- moved D35 200.1 mm to (53.7, 16.5), turned to 90 degrees
- moved D83 199.2 mm to (267.1, 16.5), turned to 90 degrees
- moved D72 198.7 mm to (265.1, 22.5), turned to 90 degrees
- moved D59 195.8 mm to (269.0, 28.5), turned to 90 degrees
- moved D82 193.5 mm to (261.2, 16.5), turned to 90 degrees
- moved D71 192.9 mm to (259.2, 22.5), turned to 90 degrees
- moved D60 191.4 mm to (79.4, 22.5), turned to 90 degrees
- moved D58 189.7 mm to (263.1, 28.5), turned to 90 degrees
- moved D81 187.8 mm to (255.2, 16.5), turned to 90 degrees
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
Commit message: Repositioning LEDs after moving keyswitches.
Parts:
- moved DS77 3.20 mm to (97.0, 122.8)
- moved DS78 3.20 mm to (152.1, 122.8)
- moved DS79 3.20 mm to (188.1, 122.8)
- moved DS80 3.20 mm to (205.1, 122.8)
- moved DS81 3.20 mm to (222.1, 122.8)
- moved DS72 2.79 mm to (256.5, 106.2)
- moved DS82 2.79 mm to (239.5, 123.2)
- moved DS83 2.79 mm to (256.5, 123.2)
- moved DS84 2.79 mm to (273.5, 123.2)
- moved DS14 2.30 mm to (256.9, 37.8)
- moved DS15 2.30 mm to (273.9, 37.8)
- moved DS30 2.30 mm to (273.9, 54.8)
- moved DS45 2.30 mm to (273.9, 71.8)
- moved DS59 2.30 mm to (273.9, 88.8)
- moved DS73 2.30 mm to (273.9, 105.8)
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Changed lines of the file:
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@@
 	(footprint "keyboard_parts:LED_RGB_SK6812Mini-E"
 		(layer "F.Cu")
-		(at 100.25 122.8)
+		(at 97.05 122.8)
 		(property "Reference" "DS77"
 			(at 0 -2.3 0)
@@
 	(footprint "keyboard_parts:LED_RGB_SK6812Mini-E"
 		(layer "F.Cu")
-		(at 225.25 122.8)
+		(at 222.05 122.8)
 		(property "Reference" "DS81"
 			(at 0 -2.3 0)
@@
 	(footprint "keyboard_parts:LED_RGB_SK6812Mini-E"
 		(layer "F.Cu")
-		(at 61.975 122.8)
+		(at 61.05 122.8)
 		(property "Reference" "DS76"
 			(at 0 -2.3 0)
@@
 	(footprint "keyboard_parts:LED_RGB_SK6812Mini-E"
 		(layer "F.Cu")
-		(at 276.25 54.8)
+		(at 273.95 54.8)
 		(property "Reference" "DS30"
 			(at 0 -2.3 0)
@@
 	(footprint "keyboard_parts:LED_RGB_SK6812Mini-E"
 		(layer "F.Cu")
-		(at 276.25 105.8)
+		(at 273.95 105.8)
 		(property "Reference" "DS73"
 			(at 0 -2.3 0)
@@
 	(footprint "keyboard_parts:LED_RGB_SK6812Mini-E"
 		(layer "F.Cu")
-		(at 259.25 37.8)
+		(at 256.95 37.8)
 		(property "Reference" "DS14"
 			(at 0 -2.3 0)
@@
 	(footprint "keyboard_parts:LED_RGB_SK6812Mini-E"
 		(layer "F.Cu")
-		(at 208.25 122.8)
+		(at 205.05 122.8)
 		(property "Reference" "DS80"
 			(at 0 -2.3 0)
@@
 	(footprint "keyboard_parts:LED_RGB_SK6812Mini-E"
 		(layer "F.Cu")
-		(at 31.875 105.8)
+		(at 32.8 105.8)
 		(property "Reference" "DS60"
 			(at 0 -2.3 0)
@@
 	(footprint "keyboard_parts:LED_RGB_SK6812Mini-E"
 		(layer "F.Cu")
-		(at 27.625 88.8)
+		(at 27.1 88.8)
 		(property "Reference" "DS46"
 			(at 0 -2.3 0)
@@
 	(footprint "keyboard_parts:LED_RGB_SK6812Mini-E"
 		(layer "F.Cu")
-		(at 191.25 122.8)
+		(at 188.05 122.8)
 		(property "Reference" "DS79"
 			(at 0 -2.3 0)
@@
 	(footprint "keyboard_parts:LED_RGB_SK6812Mini-E"
 		(layer "F.Cu")
-		(at 248.625 88.8)
+		(at 247.45 88.85)
 		(property "Reference" "DS58"
 			(at 0 -2.3 0)
@@
 	(footprint "keyboard_parts:LED_RGB_SK6812Mini-E"
 		(layer "F.Cu")
-		(at 155.25 122.8)
+		(at 152.05 122.8)
 		(property "Reference" "DS78"
 			(at 0 -2.3 0)
@@
 	(footprint "keyboard_parts:LED_RGB_SK6812Mini-E"
 		(layer "F.Cu")
-		(at 23.625 122.8)
+		(at 24.65 122.8)
 		(property "Reference" "DS74"
 			(at 0 -2.3 0)
@@
 	(footprint "keyboard_parts:LED_RGB_SK6812Mini-E"
 		(layer "F.Cu")
-		(at 276.25 71.8)
+		(at 273.95 71.8)
 		(property "Reference" "DS45"
 			(at 0 -2.3 0)
@@
 	(footprint "keyboard_parts:LED_RGB_SK6812Mini-E"
 		(layer "F.Cu")
-		(at 259.25 105.8)
+		(at 256.5 106.25)
 		(property "Reference" "DS72"
 			(at 0 -2.3 0)
@@
 	(footprint "keyboard_parts:LED_RGB_SK6812Mini-E"
 		(layer "F.Cu")
-		(at 259.25 122.8)
+		(at 256.5 123.25)
 		(property "Reference" "DS83"
 			(at 0 -2.3 0)
@@
 	(footprint "keyboard_parts:LED_RGB_SK6812Mini-E"
 		(layer "F.Cu")
-		(at 276.25 88.8)
+		(at 273.95 88.8)
 		(property "Reference" "DS59"
 			(at 0 -2.3 0)
@@
 	(footprint "keyboard_parts:LED_RGB_SK6812Mini-E"
 		(layer "F.Cu")
-		(at 42.8 122.8)
+		(at 44 122.8)
 		(property "Reference" "DS75"
 			(at 0 -2.3 0)
@@
 	(footprint "keyboard_parts:LED_RGB_SK6812Mini-E"
 		(layer "F.Cu")
-		(at 235.875 105.8)
+		(at 234.3 105.8)
 		(property "Reference" "DS71"
 			(at 0 -2.3 0)
@@
 	(footprint "keyboard_parts:LED_RGB_SK6812Mini-E"
 		(layer "F.Cu")
-		(at 242.25 122.8)
+		(at 239.5 123.25)
 		(property "Reference" "DS82"
 			(at 0 -2.3 0)
@@
 	(footprint "keyboard_parts:LED_RGB_SK6812Mini-E"
 		(layer "F.Cu")
-		(at 25.5 71.8)
+		(at 24.85 71.8)
 		(property "Reference" "DS31"
 			(at 0 -2.3 0)
@@
 	(footprint "keyboard_parts:LED_RGB_SK6812Mini-E"
 		(layer "F.Cu")
-		(at 276.25 37.8)
+		(at 273.95 37.8)
 		(property "Reference" "DS15"
 			(at 0 -2.3 0)
@@
 	(footprint "keyboard_parts:LED_RGB_SK6812Mini-E"
 		(layer "F.Cu")
-		(at 255 71.8)
+		(at 253.125 71.8)
 		(property "Reference" "DS44"
 			(at 0 -2.3 0)
@@
 	(footprint "keyboard_parts:LED_RGB_SK6812Mini-E"
 		(layer "F.Cu")
-		(at 276.25 122.8)
+		(at 273.5 123.25)
 		(property "Reference" "DS84"
 			(at 0 -2.3 0)
@@
 	(footprint "keyboard_parts:LED_RGB_SK6812Mini-E"
 		(layer "F.Cu")
-		(at 250.75 54.8)
+		(at 249.35 54.8)
 		(property "Reference" "DS29"
 			(at 0 -2.3 0)
